Commit message: created scripts to automate manipulator launching

File: Manipulator/src/manipulator_description/urdf/manipulator.urdf.xacro (robot description, xacro)
@@ -124,5 +124,10 @@
         <!-- Reasonable limits (modify as needed) -->
         <limit lower="-3.14" upper="3.14" effort="2.0" velocity="5.0"/>
-    </joint>
+        <!-- DART physics dynamics -->
+        <dynamics damping="0.1" friction="0.1"/>
+    </joint>
+    <gazebo reference="joint_1">
+        <initial_position>0.0</initial_position>
+    </gazebo>
     <link name="h_arm">
         <inertial>
@@ -156,5 +161,10 @@
         <axis xyz="1 0 0"/>
         <limit lower="-1.57" upper="1.57" effort="2.0" velocity="3.0"/>
-    </joint>
+        <!-- DART physics dynamics -->
+        <dynamics damping="0.1" friction="0.1"/>
+    </joint>
+    <gazebo reference="joint_2">
+        <initial_position>0.0</initial_position>
+    </gazebo>
     <link name="motor_3">
         <inertial>
@@ -187,5 +197,10 @@
         <axis xyz="1 0 0"/>
         <limit lower="-1.57" upper="1.57" effort="2.0" velocity="3.0"/>
-    </joint>
+        <!-- DART physics dynamics -->
+        <dynamics damping="0.1" friction="0.1"/>
+    </joint>
+    <gazebo reference="joint_3">
+        <initial_position>0.0</initial_position>
+    </gazebo>
     <link name="rod">
         <inertial>
@@ -310,5 +325,10 @@
         <axis xyz="0 1 0"/>
         <limit lower="0" upper="1.2" effort="1.0" velocity="2.0"/>
-    </joint>
+        <!-- DART physics dynamics -->
+        <dynamics damping="0.05" friction="0.05"/>
+    </joint>
+    <gazebo reference="joint_4">
+        <initial_position>0.01</initial_position>
+    </gazebo>
     <link name="gripper_R">
         <inertial>
@@ -345,4 +365,9 @@
         <limit lower="-1.2" upper="0" effort="1.0" velocity="2.0"/>
         <mimic joint="joint_4" multiplier="-1"/>
-    </joint>
+        <!-- DART physics dynamics -->
+        <dynamics damping="0.05" friction="0.05"/>
+    </joint>
+    <gazebo reference="joint_5">
+        <initial_position>-0.01</initial_position>
+    </gazebo>
 </robot>

File: Manipulator/src/manipulator_description/urdf/manipulator_gazebo.xacro (robot description, xacro)
@@ -1,10 +1,83 @@
 <?xml version="1.0"?>
 <robot xmlns:xacro="http://www.ros.org/wiki/xacro" name="manipulator">
+    <!-- Get the controller config file path using xacro -->
+    <xacro:property name="controller_config" value="$(find manipulator_controller)/config/manipulator_controllers.yaml" />
     <gazebo>
         <!-- Gazebo Harmonic (gz-sim) ROS 2 Control plugin -->
         <plugin filename="gz_ros2_control-system"
                 name="gz_ros2_control::GazeboSimROS2ControlPlugin">
-            <parameters>$(find manipulator_controller)/config/manipulator_controllers.yaml</parameters>
+            <parameters>${controller_config}</parameters>
+            <controller_manager_name>controller_manager</controller_manager_name>
         </plugin>
+    </gazebo>
+    <!-- DART Physics Engine Configuration -->
+    <!-- DART requires explicit friction and contact parameters for stable simulation -->
+    <!-- Configure friction for all links -->
+    <gazebo reference="base_plate">
+        <mu1>0.8</mu1>
+        <mu2>0.8</mu2>
+        <kp>1000000.0</kp>
+        <kd>100.0</kd>
+        <minDepth>0.001</minDepth>
+    </gazebo>
+    <gazebo reference="motor_1">
+        <mu1>0.8</mu1>
+        <mu2>0.8</mu2>
+        <kp>1000000.0</kp>
+        <kd>100.0</kd>
+    </gazebo>
+    <gazebo reference="razor_connector">
+        <mu1>0.8</mu1>
+        <mu2>0.8</mu2>
+        <kp>1000000.0</kp>
+        <kd>100.0</kd>
+    </gazebo>
+    <gazebo reference="motor_2">
+        <mu1>0.8</mu1>
+        <mu2>0.8</mu2>
+        <kp>1000000.0</kp>
+        <kd>100.0</kd>
+    </gazebo>
+    <gazebo reference="h_arm">
+        <mu1>0.8</mu1>
+        <mu2>0.8</mu2>
+        <kp>1000000.0</kp>
+        <kd>100.0</kd>
+    </gazebo>
+    <gazebo reference="motor_3">
+        <mu1>0.8</mu1>
+        <mu2>0.8</mu2>
+        <kp>1000000.0</kp>
+        <kd>100.0</kd>
+    </gazebo>
+    <gazebo reference="rod">
+        <mu1>0.8</mu1>
+        <mu2>0.8</mu2>
+        <kp>1000000.0</kp>
+        <kd>100.0</kd>
+    </gazebo>
+    <gazebo reference="gripper_base">
+        <mu1>0.8</mu1>
+        <mu2>0.8</mu2>
+        <kp>1000000.0</kp>
+        <kd>100.0</kd>
+    </gazebo>
+    <gazebo reference="motor_4">
+        <mu1>0.8</mu1>
+        <mu2>0.8</mu2>
+        <kp>1000000.0</kp>
+        <kd>100.0</kd>
+    </gazebo>
+    <gazebo reference="gripper_L">
+        <mu1>1.0</mu1>
+        <mu2>1.0</mu2>
+        <kp>1000000.0</kp>
+        <kd>100.0</kd>
+    </gazebo>
+    <gazebo reference="gripper_R">
+        <mu1>1.0</mu1>
+        <mu2>1.0</mu2>
+        <kp>1000000.0</kp>
+        <kd>100.0</kd>
     </gazebo>
 </robot>

File: Manipulator/src/manipulator_description/urdf/manipulator_ros2_control.xacro (robot description, xacro)
@@ -47,4 +47,6 @@
         </joint>
         <!-- joint_5 mimics joint_4 with multiplier=-1 in the URDF -->
+        <!-- Note: gz_ros2_control does not expose mimic joints as controllable interfaces -->
+        <!-- The mimic behavior is handled by Gazebo's physics engine via the URDF <mimic> tag -->
         <joint name="joint_5">
             <param name="mimic">joint_4</param>

Commit message: gripper corrected

File: Manipulator/src/manipulator_description/urdf/manipulator.urdf.xacro (robot description, xacro)
@@ -324,5 +324,5 @@
         <!-- Rotation about Y-axis -->
         <axis xyz="0 1 0"/>
-        <limit lower="0" upper="1.2" effort="1.0" velocity="2.0"/>
+        <limit lower="-0.001" upper="1.2" effort="1.0" velocity="2.0"/>
         <!-- DART physics dynamics -->
         <dynamics damping="0.05" friction="0.05"/>
@@ -363,5 +363,5 @@
         <!-- Rotation about Y-axis -->
         <axis xyz="0 1 0"/>
-        <limit lower="-1.2" upper="0" effort="1.0" velocity="2.0"/>
+        <limit lower="-1.2" upper="0.001" effort="1.0" velocity="2.0"/>
         <mimic joint="joint_4" multiplier="-1"/>
         <!-- DART physics dynamics -->

Commit message: integrated the hexacopter and the robot arm in Gazebo

File: Manipulator/src/manipulator_description/urdf/manipulator.urdf.xacro (robot description, xacro)
@@ -4,5 +4,6 @@
     <xacro:include filename="$(find manipulator_description)/urdf/manipulator_ros2_control.xacro"/>
     <!-- Links -->
-    <link name="world"/>
+    <!-- NOTE: world link and base_plate_fixed joint removed for aerial manipulator integration -->
+    <!-- The base_plate will be connected to hexacopter::base_link via the world file -->
     <link name="base_plate">
         <inertial>
@@ -30,9 +31,4 @@
         </collision>
     </link>
-    <joint name="base_plate_fixed" type="fixed">
-        <parent link="world"/>
-        <child link="base_plate"/>
-        <origin xyz="0 0 0.5" rpy="0 0 0"/>  <!-- Raised whole model +0.5 m along Z -->
-    </joint>
     <link name="motor_1">
         <inertial>

Commit message: gripper visuals updated

File: Manipulator/src/manipulator_description/urdf/manipulator.urdf.xacro (robot description, xacro)
@@ -287,9 +287,11 @@
         </inertial>
         <visual>
-            <origin xyz="0 0 -0.022" rpy="0 0 0"/>
-            <geometry>
-                <!-- w=10mm, h=3mm, d=60mm -->
-                <box size="0.010 0.003 0.060"/>
-            </geometry>
+            <origin xyz="-0.009 -0.002 -0.075" rpy="-${PI / 2} -${PI / 2} 0"/>
+            <geometry>
+                <mesh filename="package://manipulator_description/meshes/left_finger.STL" scale="0.0015 0.0015 0.0015"/>
+            </geometry>
+            <material name="black">
+                <color rgba="0.1 0.1 0.1 1.0"/>
+            </material>
         </visual>
         <collision>
@@ -319,9 +321,11 @@
         </inertial>
         <visual>
-            <origin xyz="0 0 -0.022" rpy="0 0 0"/>
-            <geometry>
-                <!-- w=10mm, h=3mm, d=60mm -->
-                <box size="0.010 0.003 0.060"/>
-            </geometry>
+            <origin xyz="-0.011 -0.002 -0.075" rpy="-${PI / 2} -${PI / 2} 0"/>
+            <geometry>
+                <mesh filename="package://manipulator_description/meshes/right_finger.STL" scale="0.0015 0.0015 0.0015"/>
+            </geometry>
+            <material name="black">
+                <color rgba="0.1 0.1 0.1 1.0"/>
+            </material>
         </visual>
         <collision>

Commit message: integrated the manipulator to the hexacopter and configured px4 sitl

File: Manipulator/src/manipulator_description/urdf/manipulator.urdf.xacro (robot description, xacro)
@@ -31,5 +31,5 @@
         </collision>
     </link>
-    <link name="motor_1">
+    <link name="arm_motor_1">
         <inertial>
             <origin xyz="0 0 0" rpy="0 0 0"/>
@@ -56,5 +56,5 @@
     <joint name="joint_motor_1" type="fixed">
         <parent link="base_plate"/>
-        <child link="motor_1"/>
+        <child link="arm_motor_1"/>
         <!-- Motor attached below the plate -->
         <origin xyz="0 0 -0.0245" rpy="0 0 0"/>
@@ -83,10 +83,10 @@
     </link>
     <joint name="joint_motor1_to_connector" type="fixed">
-        <parent link="motor_1"/>
+        <parent link="arm_motor_1"/>
         <child link="razor_connector"/>
         <!-- Connector sits ABOVE motor_1 -->
         <origin xyz="0.0095 0 -0.026" rpy="0 0 0"/>
     </joint>
-    <link name="motor_2">
+    <link name="arm_motor_2">
         <inertial>
             <origin xyz="0 0 0" rpy="0 0 0"/>
@@ -113,5 +113,5 @@
     <joint name="joint_1" type="revolute">
         <parent link="razor_connector"/>
-        <child link="motor_2"/>
+        <child link="arm_motor_2"/>
         <!-- Motor 2 sits ABOVE the connector -->
         <origin xyz="0 -0.010 -0.016" rpy="0 0 0"/>
@@ -150,5 +150,5 @@
     </link>
     <joint name="joint_2" type="revolute">
-        <parent link="motor_2"/>
+        <parent link="arm_motor_2"/>
         <child link="h_arm"/>
         <!-- Arm sits Below motor_2 -->
@@ -163,5 +163,5 @@
         <initial_position>0.0</initial_position>
     </gazebo>
-    <link name="motor_3">
+    <link name="arm_motor_3">
         <inertial>
             <origin xyz="0 0 -0.015" rpy="0 0 0"/>
@@ -188,5 +188,5 @@
     <joint name="joint_3" type="revolute">
         <parent link="h_arm"/>
-        <child link="motor_3"/>
+        <child link="arm_motor_3"/>
         <origin xyz="0 0 -0.106" rpy="0 0 0"/>
         <!-- Rotation around X-axis -->
@@ -224,5 +224,5 @@
     <!-- Rod fixedly connected to Motor 3 -->
     <joint name="joint_motor3_to_rod" type="fixed">
-        <parent link="motor_3"/>
+        <parent link="arm_motor_3"/>
         <child  link="rod"/>
         <!-- Rod center 0.0575 m above motor_3 center:
@@ -259,5 +259,5 @@
         <origin xyz="0 0 -0.0525" rpy="0 0 0"/>
     </joint>
-    <link name="motor_4">
+    <link name="arm_motor_4">
         <inertial>
             <origin xyz="0 0 0" rpy="0 0 0"/>
@@ -284,5 +284,5 @@
     <joint name="joint_gripperbase_to_motor4" type="fixed">
         <parent link="gripper_base"/>
-        <child  link="motor_4"/>
+        <child  link="arm_motor_4"/>
         <!-- Motor 4 mounted on top of the gripper base -->
         <origin xyz="0.027 -0.024 -0.002" rpy="0 0 0"/>

File: Manipulator/src/manipulator_description/urdf/manipulator_gazebo.xacro (robot description, xacro)
@@ -21,5 +21,5 @@
         <minDepth>0.001</minDepth>
     </gazebo>
-    <gazebo reference="motor_1">
+    <gazebo reference="arm_motor_1">
         <mu1>0.8</mu1>
         <mu2>0.8</mu2>
@@ -33,5 +33,5 @@
         <kd>100.0</kd>
     </gazebo>
-    <gazebo reference="motor_2">
+    <gazebo reference="arm_motor_2">
         <mu1>0.8</mu1>
         <mu2>0.8</mu2>
@@ -45,5 +45,5 @@
         <kd>100.0</kd>
     </gazebo>
-    <gazebo reference="motor_3">
+    <gazebo reference="arm_motor_3">
         <mu1>0.8</mu1>
         <mu2>0.8</mu2>
@@ -63,5 +63,5 @@
         <kd>100.0</kd>
     </gazebo>
-    <gazebo reference="motor_4">
+    <gazebo reference="arm_motor_4">
         <mu1>0.8</mu1>
         <mu2>0.8</mu2>
